Commit message: [Fix] adding middle and bottom link

File: pir2_description/urdf/lds/lds.urdf.xacro (robot description, xacro)
@@ -5,8 +5,62 @@
   <!--xacro:include filename="$(find pir2_description)/urdf/turtlebot3_waffle.gazebo.xacro"/-->
   <xacro:macro name="hlds_support" params="parent" >
+    <joint name="bottom_scan_joint" type="fixed">
+      <parent link="${parent}"/>
+      <child link="bottom_scan"/>
+      <origin xyz="-0.012 0 0.03" rpy="0 0 0"/>
+    </joint>
+    <link name="bottom_scan">
+      <visual>
+        <origin xyz="0 0 0" rpy="0 0 0"/>
+        <geometry>
+          <mesh filename="package://pir2_description/meshes/sensors/lds_bottom.stl" scale="0.001 0.001 0.001"/>
+        </geometry>
+        <material name="dark"/>
+      </visual>
+      <collision>
+        <origin xyz="0 0 0" rpy="0 0 0"/>
+        <geometry>
+          <cylinder length="0.0315" radius="0.055"/>
+        </geometry>
+      </collision>
+      <inertial>
+        <mass value="0.114" />
+        <origin xyz="0 0 0" />
+        <inertia ixx="0.001" ixy="0.0" ixz="0.0"
+                 iyy="0.001" iyz="0.0"
+                 izz="0.001" />
+      </inertial>
+    </link>
+    <joint name="middle_scan_joint" type="fixed">
+      <parent link="bottom_scan"/>
+      <child link="middle_scan"/>
+      <origin xyz="0.0 0 0.08" rpy="0 0 0"/>
+    </joint>
+    <link name="middle_scan">
+      <visual>
+        <origin xyz="0 0 0" rpy="0 0 0"/>
+        <geometry>
+          <mesh filename="package://pir2_description/meshes/sensors/lds_top.stl" scale="0.001 0.001 0.001"/>
+        </geometry>
+        <material name="dark"/>
+      </visual>
+      <collision>
+        <origin xyz="0 0 0" rpy="0 0 0"/>
+        <geometry>
+          <cylinder length="0.0315" radius="0.055"/>
+        </geometry>
+      </collision>
+      <inertial>
+        <mass value="0.114" />
+        <origin xyz="0 0 0" />
+        <inertia ixx="0.001" ixy="0.0" ixz="0.0"
+                 iyy="0.001" iyz="0.0"
+                 izz="0.001" />
+      </inertial>
+    </link>
     <joint name="scan_joint" type="fixed">
-      <parent link="${parent}"/>
+      <parent link="middle_scan"/>
       <child link="base_scan"/>
-      <origin xyz="-0.064 0 0.122" rpy="0 0 0"/>
+      <origin xyz="0 0 0.036" rpy="0 0 0"/>
     </joint>
     <link name="base_scan">

Commit message: [Fix] deleting hlds support links

File: pir2_description/urdf/lds/lds.urdf.xacro (robot description, xacro)
@@ -1,67 +1,10 @@
 <?xml version="1.0" ?>
 <robot name="hlds_support" xmlns:xacro="http://ros.org/wiki/xacro">
-  <!--xacro:include filename="$(find pir2_description)/urdf/common_properties.xacro"/-->
-  <!--xacro:include filename="$(find pir2_description)/urdf/materials.urdf.xacro"/-->
-  <!--xacro:include filename="$(find pir2_description)/urdf/turtlebot3_waffle.gazebo.xacro"/-->
   <xacro:include filename="$(find pir2_description)/urdf/lds/lds.gazebo.xacro"/>
-  <xacro:macro name="hlds_support" params="parent" >
-    <joint name="bottom_scan_joint" type="fixed">
+  <xacro:macro name="lds" params="parent" >
+    <joint name="scan_joint" type="fixed">
       <parent link="${parent}"/>
-      <child link="bottom_scan"/>
-      <origin xyz="-0.012 0 0.03" rpy="0 0 0"/>
-    </joint>
-    <link name="bottom_scan">
-      <visual>
-        <origin xyz="0 0 0" rpy="0 0 0"/>
-        <geometry>
-          <mesh filename="package://pir2_description/meshes/sensors/lds_bottom.stl" scale="0.001 0.001 0.001"/>
-        </geometry>
-        <material name="dark"/>
-      </visual>
-      <collision>
-        <origin xyz="0 0 0" rpy="0 0 0"/>
-        <geometry>
-          <cylinder length="0.0315" radius="0.055"/>
-        </geometry>
-      </collision>
-      <inertial>
-        <mass value="0.114" />
-        <origin xyz="0 0 0" />
-        <inertia ixx="0.001" ixy="0.0" ixz="0.0"
-                 iyy="0.001" iyz="0.0"
-                 izz="0.001" />
-      </inertial>
-    </link>
-    <joint name="middle_scan_joint" type="fixed">
-      <parent link="bottom_scan"/>
-      <child link="middle_scan"/>
-      <origin xyz="0.0 0 0.08" rpy="0 0 0"/>
-    </joint>
-    <link name="middle_scan">
-      <visual>
-        <origin xyz="0 0 0" rpy="0 0 0"/>
-        <geometry>
-          <mesh filename="package://pir2_description/meshes/sensors/lds_top.stl" scale="0.001 0.001 0.001"/>
-        </geometry>
-        <material name="dark"/>
-      </visual>
-      <collision>
-        <origin xyz="0 0 0" rpy="0 0 0"/>
-        <geometry>
-          <cylinder length="0.0315" radius="0.055"/>
-        </geometry>
-      </collision>
-      <inertial>
-        <mass value="0.114" />
-        <origin xyz="0 0 0" />
-        <inertia ixx="0.001" ixy="0.0" ixz="0.0"
-                 iyy="0.001" iyz="0.0"
-                 izz="0.001" />
-      </inertial>
-    </link>
-    <joint name="scan_joint" type="fixed">
-      <parent link="middle_scan"/>
       <child link="base_scan"/>
-      <origin xyz="0 0 0.036" rpy="0 0 0"/>
+      <origin xyz="-0.01 0 0.023" rpy="0 0 0"/>
     </joint>
     <link name="base_scan">
