Commit message: [Fix] collision values

File: pir2_description/urdf/body/top.urdf.xacro (robot description, xacro)
@@ -18,5 +18,5 @@
         <origin xyz="0 0 0" rpy="0 0 0"/>
         <geometry>
-          <cylinder length="0.05" radius="0.285"/>
+          <cylinder length="0.02" radius="0.14"/>
         </geometry>
       </collision>

File: pir2_description/urdf/head/head.urdf.xacro (robot description, xacro)
@@ -17,13 +17,19 @@
           <mesh filename="package://pir2_description/meshes/head/pan_frame.stl" scale="0.001 0.001 0.001"/>
         </geometry>
-        <material name="gray"/>
+        <material name="grey"/>
       </visual>
+      <collision>
+        <origin xyz="-0.015 0 0" rpy="0 0 0"/>
+        <geometry>
+           <box size="0.06 0.06 0.05"/>
+        </geometry>
+      </collision>
      <inertial>
        <origin xyz="0 0 0" rpy="0 0 0"/>
-       <mass value="0.78"/>
+       <mass value="0.3"/>
        <inertia
-	    ixx="0.00190" ixy="0.0" ixz="0.0"
-	    iyy="0.00202" iyz="0.0"
-	    izz="0.00152"/>
+  	    ixx="0.00190" ixy="0.0" ixz="0.0"
+  	    iyy="0.00202" iyz="0.0"
+  	    izz="0.00152"/>
      </inertial>
     </link>
@@ -43,14 +49,20 @@
           <mesh filename="package://pir2_description/meshes/head/tilt_frame.stl" scale="0.001 0.001 0.001"/>
         </geometry>
-        <material name="gray"/>
+        <material name="grey"/>
       </visual>
-     <inertial>
-       <origin xyz="0 0 0.0515" rpy="0 0 0"/>
-       <mass value="0.78"/>
-       <inertia
-      ixx="0.00190" ixy="0.0" ixz="0.0"
-      iyy="0.00202" iyz="0.0"
-      izz="0.00152"/>
-     </inertial>
+      <collision>
+        <origin xyz="0 0 0.018" rpy="0 0 0"/>
+        <geometry>
+          <box size="0.04 0.04 0.03"/>
+        </geometry>
+      </collision>
+      <inertial>
+        <origin xyz="-0.015 0 0" rpy="0 0 0"/>
+        <mass value="0.78"/>
+        <inertia
+          ixx="0.00190" ixy="0.0" ixz="0.0"
+          iyy="0.00202" iyz="0.0"
+          izz="0.00152"/>
+      </inertial>
     </link>
     <joint name="tilt_joint" type="revolute">
@@ -66,17 +78,22 @@
         <origin xyz="0 0 -0.0245" rpy="0 0 0" />
         <geometry>
-          <!--box size="0.07 0.085 0.065" /-->
           <mesh filename="package://pir2_description/meshes/head/yaw_plate.stl" scale="0.001 0.001 0.001"/>
         </geometry>
-        <material name="gray"/>
+        <material name="grey"/>
       </visual>
-     <inertial>
-       <origin xyz="0 -0.0245 0" rpy="0 0 0"/>
-       <mass value="0.78"/>
-       <inertia
-      ixx="0.00190" ixy="0.0" ixz="0.0"
-      iyy="0.00202" iyz="0.0"
-      izz="0.00152"/>
-     </inertial>
+      <collision>
+        <origin xyz="0.035 0 -0.025" rpy="0 0 0"/>
+        <geometry>
+          <box size="0.004 0.18 0.06"/>
+        </geometry>
+      </collision>
+      <inertial>
+        <origin xyz="0 -0.0245 0" rpy="0 0 0"/>
+        <mass value="0.78"/>
+        <inertia
+          ixx="0.00190" ixy="0.0" ixz="0.0"
+          iyy="0.00202" iyz="0.0"
+          izz="0.00152"/>
+      </inertial>
     </link>
     <joint name="yaw_plate_to_dxl_joint" type="fixed">
@@ -89,17 +106,22 @@
         <origin xyz="0 0 0" rpy="0 0 0" />
         <geometry>
-          <!--box size="0.07 0.085 0.065" /-->
           <mesh filename="package://pir2_description/meshes/head/yaw_frame.stl" scale="0.001 0.001 0.001"/>
         </geometry>
-        <material name="gray"/>
+        <material name="grey"/>
       </visual>
-     <inertial>
-       <origin xyz="0 -0.0245 0" rpy="0 0 0"/>
-       <mass value="0.78"/>
-       <inertia
-      ixx="0.00190" ixy="0.0" ixz="0.0"
-      iyy="0.00202" iyz="0.0"
-      izz="0.00152"/>
-     </inertial>
+      <collision>
+        <origin xyz="-0.013 0 -0.015" rpy="0 0 0"/>
+        <geometry>
+          <box size="0.035 0.053 0.054"/>
+        </geometry>
+      </collision>
+      <inertial>
+        <origin xyz="0 -0.0245 0" rpy="0 0 0"/>
+        <mass value="0.78"/>
+        <inertia
+         ixx="0.00190" ixy="0.0" ixz="0.0"
+         iyy="0.00202" iyz="0.0"
+         izz="0.00152"/>
+      </inertial>
     </link>
     <joint name="yaw_joint" type="revolute">
@@ -118,14 +140,20 @@
           <mesh filename="package://pir2_description/meshes/head/display_frame.stl" scale="0.001 0.001 0.001"/>
         </geometry>
-        <material name="gray"/>
+        <material name="grey"/>
       </visual>
-     <inertial>
-       <origin xyz="0 0 0" rpy="0 0 0"/>
-       <mass value="0.78"/>
-       <inertia
-      ixx="0.00190" ixy="0.0" ixz="0.0"
-      iyy="0.00202" iyz="0.0"
-      izz="0.00152"/>
-     </inertial>
+      <collision>
+        <origin xyz="0 0 0" rpy="0 0 0"/>
+        <geometry>
+          <box size="0.16 0.26 0.004"/>
+        </geometry>
+      </collision>
+      <inertial>
+        <origin xyz="0 0 0" rpy="0 0 0"/>
+        <mass value="0.78"/>
+        <inertia
+          ixx="0.00190" ixy="0.0" ixz="0.0"
+          iyy="0.00202" iyz="0.0"
+          izz="0.00152"/>
+       </inertial>
     </link>
   </xacro:macro>
