Commit message: [Add] pan_support link

File: pir2_description/urdf/body/middle.urdf.xacro (robot description, xacro)
@@ -23,5 +23,5 @@
       <!-- <inertial>
         <origin xyz="0 0 0" rpy="0 0 0"/>
-        <mass value="0.4"/>
+        <mass value="0.8"/>
         <inertia ixx="0.008" ixy="0" ixz="0"
                  iyy="0.008" iyz="0"

File: pir2_description/urdf/body/top.urdf.xacro (robot description, xacro)
@@ -23,8 +23,8 @@
       <!-- <inertial>
         <origin xyz="0 0 0" rpy="0 0 0"/>
-        <mass value="0.4"/>
-        <inertia ixx="0.008" ixy="0" ixz="0"
-                 iyy="0.008" iyz="0"
-                 izz="0.016" />
+        <mass value="0.7"/>
+        <inertia ixx="0.0034" ixy="0" ixz="0"
+                 iyy="0.0034" iyz="0"
+                 izz="0.0068" />
       </inertial> -->
     </link>

File: pir2_description/urdf/head/head.urdf.xacro (robot description, xacro)
@@ -5,4 +5,18 @@
   <xacro:macro name="head_frame" params="parent angle">
     <xacro:property name="yaw_angle" value="${-angle}"/>
+    <joint name="pan_support_joint" type="fixed">
+      <origin xyz="0 0 0.0015 " rpy="0 0 0" />
+      <parent link="${parent}"/>
+      <child link="pan_support_link"/>
+    </joint>
+    <link name="pan_support_link" >
+      <visual>
+        <origin xyz="0 0 0" rpy="0 0 0" />
+        <geometry>
+          <mesh filename="package://pir2_description/meshes/head/pan_support.stl" scale="0.001 0.001 0.001"/>
+        </geometry>
+        <material name="grey"/>
+      </visual>
+    </link>
     <joint name="head_base_joint" type="fixed">
       <origin xyz="0 0 0.0316 " rpy="0 0 0" />
@@ -26,10 +40,10 @@
       </collision>
      <inertial>
-       <origin xyz="0 0 0" rpy="0 0 0"/>
-       <mass value="0.3"/>
+       <origin xyz="-0.015 0 0" rpy="0 0 0"/>
+       <mass value="0.2"/>
        <inertia
-  	    ixx="0.00190" ixy="0.0" ixz="0.0"
-  	    iyy="0.00202" iyz="0.0"
-  	    izz="0.00152"/>
+  	    ixx="0.0001" ixy="0.0" ixz="0.0"
+  	    iyy="0.00012" iyz="0.0"
+  	    izz="0.0001"/>
      </inertial>
     </link>
@@ -58,10 +72,10 @@
       </collision>
       <inertial>
-        <origin xyz="-0.015 0 0" rpy="0 0 0"/>
-        <mass value="0.78"/>
+        <origin xyz="0 0 0.018" rpy="0 0 0"/>
+        <mass value="0.3"/>
         <inertia
-          ixx="0.00190" ixy="0.0" ixz="0.0"
-          iyy="0.00202" iyz="0.0"
-          izz="0.00152"/>
+          ixx="0.0000625" ixy="0.0" ixz="0.0"
+          iyy="0.00008" iyz="0.0"
+          izz="0.0000625"/>
       </inertial>
     </link>
@@ -89,10 +103,10 @@
       </collision>
       <inertial>
-        <origin xyz="0 -0.0245 0" rpy="0 0 0"/>
-        <mass value="0.78"/>
+        <origin xyz="0.035 0 -0.025" rpy="0 0 0"/>
+        <mass value="0.4"/>
         <inertia
-          ixx="0.00190" ixy="0.0" ixz="0.0"
-          iyy="0.00202" iyz="0.0"
-          izz="0.00152"/>
+          ixx="0.032" ixy="0.0" ixz="0.0"
+          iyy="0.0010" iyz="0.0"
+          izz="0.0012"/>
       </inertial>
     </link>
@@ -117,10 +131,10 @@
       </collision>
       <inertial>
-        <origin xyz="0 -0.0245 0" rpy="0 0 0"/>
-        <mass value="0.78"/>
+        <origin xyz="-0.013 0 -0.015" rpy="0 0 0"/>
+        <mass value="0.2"/>
         <inertia
-         ixx="0.00190" ixy="0.0" ixz="0.0"
-         iyy="0.00202" iyz="0.0"
-         izz="0.00152"/>
+         ixx="0.0028" ixy="0.0" ixz="0.0"
+         iyy="0.0012" iyz="0.0"
+         izz="0.0012"/>
       </inertial>
     </link>
@@ -150,9 +164,9 @@
       <inertial>
         <origin xyz="0 0 0" rpy="0 0 0"/>
-        <mass value="0.78"/>
+        <mass value="0.1"/>
         <inertia
-          ixx="0.00190" ixy="0.0" ixz="0.0"
-          iyy="0.00202" iyz="0.0"
-          izz="0.00152"/>
+          ixx="0.00057" ixy="0.0" ixz="0.0"
+          iyy="0.00077" iyz="0.0"
+          izz="0.025"/>
        </inertial>
     </link>
