Commit message: [Edit] wheel inertial value

File: pir2_description/urdf/body/bottom.gazebo.xacro (robot description, xacro)
@@ -4,25 +4,3 @@
     <material>Gazebo/DarkGrey</material>
   </gazebo>
-  <gazebo>
-    <plugin name="pir2_robot_frame_controller" filename="libgazebo_ros_diff_drive.so">
-      <commandTopic>cmd_vel</commandTopic>
-      <odometryTopic>odom</odometryTopic>
-      <odometryFrame>odom</odometryFrame>
-      <odometrySource>world</odometrySource>
-      <publishOdomTF>true</publishOdomTF>
-      <robotBaseFrame>base_footprint</robotBaseFrame>
-      <publishWheelTF>false</publishWheelTF>
-      <publishTf>true</publishTf>
-      <publishWheelJointState>true</publishWheelJointState>
-      <legacyMode>false</legacyMode>
-      <updateRate>30</updateRate>
-      <leftJoint>wheel_left_joint</leftJoint>
-      <rightJoint>wheel_right_joint</rightJoint>
-      <wheelSeparation>0.287</wheelSeparation>
-      <wheelDiameter>0.120</wheelDiameter>
-      <wheelAcceleration>1</wheelAcceleration>
-      <wheelTorque>10</wheelTorque>
-      <rosDebugLevel>na</rosDebugLevel>
-    </plugin>
-  </gazebo>
 </robot>

File: pir2_description/urdf/wheels/wheel.gazebo.xacro (robot description, xacro)
@@ -36,6 +36,6 @@
       <leftJoint>wheel_left_joint</leftJoint>
       <rightJoint>wheel_right_joint</rightJoint>
-      <wheelSeparation>0.287</wheelSeparation>
-      <wheelDiameter>0.120</wheelDiameter>
+      <wheelSeparation>0.58</wheelSeparation>
+      <wheelDiameter>0.216</wheelDiameter>
       <wheelAcceleration>1</wheelAcceleration>
       <wheelTorque>10</wheelTorque>

File: pir2_description/urdf/wheels/wheel.urdf.xacro (robot description, xacro)
@@ -25,8 +25,8 @@
       <inertial>
         <origin xyz="0 0 0" />
-        <mass value="0.2" />
-        <inertia ixx="1.1175580e-05" ixy="-4.2369783e-11" ixz="-5.9381719e-09"
-                 iyy="1.1192413e-05" iyz="-1.4400107e-11"
-                 izz="2.0712558e-05" />
+        <mass value="0.230446843750" />
+        <inertia ixx="1" ixy="0" ixz="0"
+                 iyy="1" iyz="0"
+                 izz="1" />
         </inertial>
     </link>
@@ -53,8 +53,8 @@
       <inertial>
         <origin xyz="0 0 0" />
-        <mass value="0.2" />
-        <inertia ixx="1.1175580e-05" ixy="-4.2369783e-11" ixz="-5.9381719e-09"
-                 iyy="1.1192413e-05" iyz="-1.4400107e-11"
-                 izz="2.0712558e-05" />
+        <mass value="2" />
+        <inertia ixx="1" ixy="0" ixz="0"
+                 iyy="1" iyz="0"
+                 izz="1" />
         </inertial>
     </link>

Commit message: [Edit] link color

File: pir2_description/urdf/body/bottom.gazebo.xacro (robot description, xacro)
@@ -2,5 +2,5 @@
 <robot name="pir2_sim" xmlns:xacro="http://ros.org/wiki/xacro">
   <gazebo reference="base_link">
-    <material>DarkGrey</material>
+    <material>LightGrey</material>
   </gazebo>
   <gazebo>

File: pir2_description/urdf/body/bottom.urdf.xacro (robot description, xacro)
@@ -1,4 +1,5 @@
 <?xml version="1.0" ?>
 <robot name="bottom_frame" xmlns:xacro="http://ros.org/wiki/xacro">
+  <xacro:include filename="$(find pir2_description)/urdf/body/bottom.gazebo.xacro"/>
   <xacro:macro name="bottom_frame" params="parent" >
     <link name="base_footprint"/>

File: pir2_description/urdf/head/head.gazebo.xacro (robot description, xacro)
@@ -5,20 +5,25 @@
     <mu1>0.2</mu1>
     <mu2>0.2</mu2>
-    <material>Gazebo/LightGrey</material>
+    <material>Gazebo/Grey</material>
+  </gazebo>
+  <gazebo reference="pan_support_link">
+    <mu1>0.2</mu1>
+    <mu2>0.2</mu2>
+    <material>Gazebo/Green</material>
   </gazebo>
   <gazebo reference="tilt_link">
     <mu1>0.2</mu1>
     <mu2>0.2</mu2>
-    <material>Gazebo/LightGrey</material>
+    <material>Gazebo/Grey</material>
   </gazebo>
   <gazebo reference="pan_link">
     <mu1>0.2</mu1>
     <mu2>0.2</mu2>
-    <material>Gazebo/LightGrey</material>
+    <material>Gazebo/Grey</material>
   </gazebo>
   <gazebo reference="yaw_link">
     <mu1>0.2</mu1>
     <mu2>0.2</mu2>
-    <material>Gazebo/LightGrey</material>
+    <material>Gazebo/FlatBlack</material>
   </gazebo>
 </xacro:macro>

File: pir2_description/urdf/wheels/wheel.gazebo.xacro (robot description, xacro)
@@ -9,5 +9,5 @@
     <maxVel>0.1</maxVel>
     <fdir1>1 0 0</fdir1>
-    <material>Gazebo/LightGrey</material>
+    <material>LightGrey</material>
   </gazebo>
   <gazebo reference="wheel_right_link">
@@ -19,5 +19,5 @@
     <maxVel>0.1</maxVel>
     <fdir1>1 0 0</fdir1>
-    <material>Gazebo/LightGrey</material>
+    <material>LightGrey</material>
   </gazebo>
   <gazebo>
