Commit message: [Fix] collision parameters

File: pir2_description/urdf/body/bottom.urdf.xacro (robot description, xacro)
@@ -2,4 +2,5 @@
 <robot name="pir2" xmlns:xacro="http://ros.org/wiki/xacro">
   <xacro:include filename="$(find pir2_description)/urdf/common_properties.xacro"/>
+  <xacro:include filename="$(find pir2_description)/urdf/wheels/wheel.urdf.xacro"/>
   <!--xacro:include filename="$(find pir2_description)/urdf/bottom.urdf.xacro"/-->
   <link name="base_footprint"/>
@@ -7,5 +8,5 @@
     <parent link="base_footprint"/>
     <child link="base_link" />
-    <origin xyz="0 0 0.088" rpy="0 0 0"/>
+    <origin xyz="0 0 0.086" rpy="0 0 0"/>
   </joint>
   <link name="base_link">
@@ -31,3 +32,59 @@
     </inertial>
   </link>
+  <joint name="caster_front_joint" type="fixed">
+    <parent link="base_link"/>
+    <child link="caster_front_link"/>
+    <origin xyz="0.2 0 0" rpy="0 0 0"/>
+  </joint>
+  <link name="caster_front_link">
+    <visual>
+      <origin xyz="0 0 0" rpy="0 0 0"/>
+      <geometry>
+        <!--box size="0.07 0.085 0.065"/-->
+        <mesh filename="package://pir2_description/meshes/wheels/caster.stl" scale="0.001 0.001 0.001"/>
+      </geometry>
+      <material name="dark"/>
+    </visual>
+    <collision>
+      <origin xyz="0 0.001 0" rpy="0 0 0"/>
+      <geometry>
+        <box size="0.030 0.009 0.020"/>
+      </geometry>
+    </collision>
+    <inertial>
+      <origin xyz="0 0 0" />
+      <mass value="0.005" />
+      <inertia ixx="0.001" ixy="0.0" ixz="0.0"
+               iyy="0.001" iyz="0.0"
+               izz="0.001" />
+    </inertial>
+  </link>
+  <joint name="caster_rear_joint" type="fixed">
+    <parent link="base_link"/>
+    <child link="caster_rear_link"/>
+    <origin xyz="-0.2 0 0" rpy="0 0 0"/>
+  </joint>
+  <link name="caster_rear_link">
+    <visual>
+      <origin xyz="0 0 0" rpy="0 0 0"/>
+      <geometry>
+        <!--box size="0.07 0.085 0.065"/-->
+        <mesh filename="package://pir2_description/meshes/wheels/caster.stl" scale="0.001 0.001 0.001"/>
+      </geometry>
+      <material name="dark"/>
+    </visual>
+    <collision>
+      <origin xyz="0 0.001 0" rpy="0 0 0"/>
+      <geometry>
+        <box size="0.030 0.009 0.020"/>
+      </geometry>
+    </collision>
+    <inertial>
+      <origin xyz="0 0 0" />
+      <mass value="0.005" />
+      <inertia ixx="0.001" ixy="0.0" ixz="0.0"
+               iyy="0.001" iyz="0.0"
+               izz="0.001" />
+    </inertial>
+  </link>
 </robot>

Commit message: [Fix] adding gazebo xacro files

File: pir2_description/urdf/body/bottom.urdf.xacro (robot description, xacro)
@@ -2,4 +2,5 @@
 <robot name="pir2" xmlns:xacro="http://ros.org/wiki/xacro">
   <xacro:include filename="$(find pir2_description)/urdf/common_properties.xacro"/>
+  <xacro:include filename="$(find pir2_description)/urdf/body/bottom.gazebo.xacro"/>
   <xacro:include filename="$(find pir2_description)/urdf/wheels/wheel.urdf.xacro"/>
   <xacro:include filename="$(find pir2_description)/urdf/lds/lds.urdf.xacro"/>
@@ -19,7 +20,7 @@
     </visual>
     <collision>
-      <origin xyz="0 0 0.04" rpy="0 0 0"/>
+      <origin xyz="0 0 0" rpy="0 0 0"/>
       <geometry>
-        <box size="0.266 0.266 0.094"/>
+        <cylinder length="0.05" radius="0.285"/>
       </geometry>
     </collision>
@@ -47,7 +48,7 @@
     </visual>
     <collision>
-      <origin xyz="0 0.001 0" rpy="0 0 0"/>
+      <origin xyz="0 0.001 -0.025" rpy="0 0 0"/>
       <geometry>
-        <box size="0.030 0.009 0.020"/>
+        <box size="0.060 0.02 0.11"/>
       </geometry>
     </collision>
@@ -75,7 +76,7 @@
     </visual>
     <collision>
-      <origin xyz="0 0.001 0" rpy="0 0 0"/>
+      <origin xyz="0 0.001 -0.025" rpy="0 0 0"/>
       <geometry>
-        <box size="0.030 0.009 0.020"/>
+        <box size="0.060 0.02 0.11"/>
       </geometry>
     </collision>

File: pir2_description/urdf/lds/lds.urdf.xacro (robot description, xacro)
@@ -4,4 +4,5 @@
   <!--xacro:include filename="$(find pir2_description)/urdf/materials.urdf.xacro"/-->
   <!--xacro:include filename="$(find pir2_description)/urdf/turtlebot3_waffle.gazebo.xacro"/-->
+  <xacro:include filename="$(find pir2_description)/urdf/lds/lds.gazebo.xacro"/>
   <xacro:macro name="hlds_support" params="parent" >
     <joint name="bottom_scan_joint" type="fixed">

File: pir2_description/urdf/wheels/wheel.urdf.xacro (robot description, xacro)
@@ -1,4 +1,5 @@
 <?xml version="1.0" ?>
 <robot name="pir2_wheel" xmlns:xacro="http://ros.org/wiki/xacro">
+  <xacro:include filename="$(find pir2_description)/urdf/wheels/wheel.gazebo.xacro"/>
   <!--xacro:include filename="$(find turtlebot3_description)/urdf/turtlebot3_waffle.gazebo.xacro"/-->
   <joint name="wheel_left_joint" type="continuous">
@@ -19,5 +20,5 @@
       <origin xyz="0 0 0" rpy="0 0 0"/>
       <geometry>
-        <cylinder length="0.018" radius="0.21"/>
+        <cylinder length="0.018" radius="0.108"/>
       </geometry>
     </collision>
@@ -47,5 +48,5 @@
       <origin xyz="0 0 0" rpy="0 0 0"/>
       <geometry>
-        <cylinder length="0.018" radius="0.21"/>
+        <cylinder length="0.018" radius="0.108"/>
       </geometry>
     </collision>

Commit message: [Fix] delete include xacro files

File: pir2_description/urdf/body/bottom.urdf.xacro (robot description, xacro)
@@ -1,92 +1,89 @@
 <?xml version="1.0" ?>
-<robot name="pir2" xmlns:xacro="http://ros.org/wiki/xacro">
-  <xacro:include filename="$(find pir2_description)/urdf/common_properties.xacro"/>
-  <xacro:include filename="$(find pir2_description)/urdf/body/bottom.gazebo.xacro"/>
-  <xacro:include filename="$(find pir2_description)/urdf/wheels/wheel.urdf.xacro"/>
-  <xacro:include filename="$(find pir2_description)/urdf/lds/lds.urdf.xacro"/>
-  <link name="base_footprint"/>
-  <joint name="base_joint" type="fixed">
-    <parent link="base_footprint"/>
-    <child link="base_link" />
-    <origin xyz="0 0 0.086" rpy="0 0 0"/>
-  </joint>
-  <link name="base_link">
-    <visual>
-      <origin xyz="0 0 0.0" rpy="0 0 0"/>
-      <geometry>
-        <mesh filename="package://pir2_description/meshes/base/bottom_frame.stl" scale="0.001 0.001 0.001"/>
-      </geometry>
-      <material name="light_black"/>
-    </visual>
-    <collision>
-      <origin xyz="0 0 0" rpy="0 0 0"/>
-      <geometry>
-        <cylinder length="0.05" radius="0.285"/>
-      </geometry>
-    </collision>
-    <inertial>
-      <origin xyz="0 0 0" rpy="0 0 0"/>
-      <mass value="1.3729096e+00"/>
-      <inertia ixx="8.7002718e-03" ixy="-4.7576583e-05" ixz="1.1160499e-04"
-               iyy="8.6195418e-03" iyz="-3.5422299e-06"
-               izz="1.4612727e-02" />
-    </inertial>
-  </link>
-  <joint name="caster_front_joint" type="fixed">
-    <parent link="base_link"/>
-    <child link="caster_front_link"/>
-    <origin xyz="0.2 0 0" rpy="0 0 0"/>
-  </joint>
-  <link name="caster_front_link">
-    <visual>
-      <origin xyz="0 0 0" rpy="0 0 0"/>
-      <geometry>
-        <!--box size="0.07 0.085 0.065"/-->
-        <mesh filename="package://pir2_description/meshes/wheels/caster.stl" scale="0.001 0.001 0.001"/>
-      </geometry>
-      <material name="dark"/>
-    </visual>
-    <collision>
-      <origin xyz="0 0.001 -0.025" rpy="0 0 0"/>
-      <geometry>
-        <box size="0.060 0.02 0.11"/>
-      </geometry>
-    </collision>
-    <inertial>
-      <origin xyz="0 0 0" />
-      <mass value="0.005" />
-      <inertia ixx="0.001" ixy="0.0" ixz="0.0"
-               iyy="0.001" iyz="0.0"
-               izz="0.001" />
-    </inertial>
-  </link>
-  <joint name="caster_rear_joint" type="fixed">
-    <parent link="base_link"/>
-    <child link="caster_rear_link"/>
-    <origin xyz="-0.2 0 0" rpy="0 0 0"/>
-  </joint>
-  <link name="caster_rear_link">
-    <visual>
-      <origin xyz="0 0 0" rpy="0 0 0"/>
-      <geometry>
-        <!--box size="0.07 0.085 0.065"/-->
-        <mesh filename="package://pir2_description/meshes/wheels/caster.stl" scale="0.001 0.001 0.001"/>
-      </geometry>
-      <material name="dark"/>
-    </visual>
-    <collision>
-      <origin xyz="0 0.001 -0.025" rpy="0 0 0"/>
-      <geometry>
-        <box size="0.060 0.02 0.11"/>
-      </geometry>
-    </collision>
-    <inertial>
-      <origin xyz="0 0 0" />
-      <mass value="0.005" />
-      <inertia ixx="0.001" ixy="0.0" ixz="0.0"
-               iyy="0.001" iyz="0.0"
-               izz="0.001" />
-    </inertial>
-  </link>
-<xacro:hlds_support parent="base_link" />
+<robot name="bottom_frame" xmlns:xacro="http://ros.org/wiki/xacro">
+  <xacro:macro name="bottom_frame" params="parent" >
+    <link name="base_footprint"/>
+    <joint name="base_joint" type="fixed">
+      <parent link="base_footprint"/>
+      <child link="base_link" />
+      <origin xyz="0 0 0.086" rpy="0 0 0"/>
+    </joint>
+    <link name="base_link">
+      <visual>
+        <origin xyz="0 0 0.0" rpy="0 0 0"/>
+        <geometry>
+          <mesh filename="package://pir2_description/meshes/base/bottom_frame.stl" scale="0.001 0.001 0.001"/>
+        </geometry>
+        <material name="light_black"/>
+      </visual>
+      <collision>
+        <origin xyz="0 0 0" rpy="0 0 0"/>
+        <geometry>
+          <cylinder length="0.05" radius="0.285"/>
+        </geometry>
+      </collision>
+      <inertial>
+        <origin xyz="0 0 0" rpy="0 0 0"/>
+        <mass value="1.3729096e+00"/>
+        <inertia ixx="8.7002718e-03" ixy="-4.7576583e-05" ixz="1.1160499e-04"
+                 iyy="8.6195418e-03" iyz="-3.5422299e-06"
+                 izz="1.4612727e-02" />
+      </inertial>
+    </link>
+    <joint name="caster_front_joint" type="fixed">
+      <parent link="base_link"/>
+      <child link="caster_front_link"/>
+      <origin xyz="0.2 0 0" rpy="0 0 0"/>
+    </joint>
+    <link name="caster_front_link">
+      <visual>
+        <origin xyz="0 0 0" rpy="0 0 0"/>
+        <geometry>
+          <!--box size="0.07 0.085 0.065"/-->
+          <mesh filename="package://pir2_description/meshes/wheels/caster.stl" scale="0.001 0.001 0.001"/>
+        </geometry>
+        <material name="dark"/>
+      </visual>
+      <collision>
+        <origin xyz="0 0.001 -0.025" rpy="0 0 0"/>
+        <geometry>
+          <box size="0.060 0.02 0.11"/>
+        </geometry>
+      </collision>
+      <inertial>
+        <origin xyz="0 0 0" />
+        <mass value="0.005" />
+        <inertia ixx="0.001" ixy="0.0" ixz="0.0"
+                 iyy="0.001" iyz="0.0"
+                 izz="0.001" />
+      </inertial>
+    </link>
+    <joint name="caster_rear_joint" type="fixed">
+      <parent link="base_link"/>
+      <child link="caster_rear_link"/>
+      <origin xyz="-0.2 0 0" rpy="0 0 0"/>
+    </joint>
+    <link name="caster_rear_link">
+      <visual>
+        <origin xyz="0 0 0" rpy="0 0 0"/>
+        <geometry>
+          <!--box size="0.07 0.085 0.065"/-->
+          <mesh filename="package://pir2_description/meshes/wheels/caster.stl" scale="0.001 0.001 0.001"/>
+        </geometry>
+        <material name="dark"/>
+      </visual>
+      <collision>
+        <origin xyz="0 0.001 -0.025" rpy="0 0 0"/>
+        <geometry>
+          <box size="0.060 0.02 0.11"/>
+        </geometry>
+      </collision>
+      <inertial>
+        <origin xyz="0 0 0" />
+        <mass value="0.005" />
+        <inertia ixx="0.001" ixy="0.0" ixz="0.0"
+                 iyy="0.001" iyz="0.0"
+                 izz="0.001" />
+      </inertial>
+    </link>
+  </xacro:macro>
 </robot>

Commit message: [Edit] collision and inertia

File: pir2_description/urdf/body/bottom.urdf.xacro (robot description, xacro)
@@ -47,5 +47,5 @@
         <origin xyz="0 0.001 -0.025" rpy="0 0 0"/>
         <geometry>
-          <box size="0.060 0.02 0.11"/>
+          <sphere radius="0.05"/>
         </geometry>
       </collision>
@@ -75,5 +75,5 @@
         <origin xyz="0 0.001 -0.025" rpy="0 0 0"/>
         <geometry>
-          <box size="0.060 0.02 0.11"/>
+          <sphere radius="0.05"/>
         </geometry>
       </collision>

File: pir2_description/urdf/body/lds_plate.urdf.xacro (robot description, xacro)
@@ -18,13 +18,13 @@
         <origin xyz="0 0 0" rpy="0 0 0"/>
         <geometry>
-          <cylinder length="0.05" radius="0.285"/>
+          <cylinder length="0.03" radius="0.08"/>
         </geometry>
       </collision>
       <inertial>
         <origin xyz="0 0 0" rpy="0 0 0"/>
-        <mass value="1.3729096e+00"/>
-        <inertia ixx="8.7002718e-03" ixy="-4.7576583e-05" ixz="1.1160499e-04"
-                 iyy="8.6195418e-03" iyz="-3.5422299e-06"
-                 izz="1.4612727e-02" />
+        <mass value="0.50"/>
+        <inertia ixx="1e-3" ixy="0" ixz="0"
+                 iyy="1e-3" iyz="-0"
+                 izz="1e-3" />
       </inertial>
     </link>

File: pir2_description/urdf/body/middle.urdf.xacro (robot description, xacro)
@@ -23,8 +23,8 @@
       <inertial>
         <origin xyz="0 0 0" rpy="0 0 0"/>
-        <mass value="1.3729096e+00"/>
-        <inertia ixx="8.7002718e-03" ixy="-4.7576583e-05" ixz="1.1160499e-04"
-                 iyy="8.6195418e-03" iyz="-3.5422299e-06"
-                 izz="1.4612727e-02" />
+        <mass value="0.50"/>
+        <inertia ixx="1e-3" ixy="0" ixz="0"
+                 iyy="1e-3" iyz="0"
+                 izz="1e-3" />
       </inertial>
     </link>

File: pir2_description/urdf/wheels/wheel.urdf.xacro (robot description, xacro)
@@ -25,5 +25,5 @@
       <inertial>
         <origin xyz="0 0 0" />
-        <mass value="2.8498940e-02" />
+        <mass value="0.2" />
         <inertia ixx="1.1175580e-05" ixy="-4.2369783e-11" ixz="-5.9381719e-09"
                  iyy="1.1192413e-05" iyz="-1.4400107e-11"
@@ -53,5 +53,5 @@
       <inertial>
         <origin xyz="0 0 0" />
-        <mass value="2.8498940e-02" />
+        <mass value="0.2" />
         <inertia ixx="1.1175580e-05" ixy="-4.2369783e-11" ixz="-5.9381719e-09"
                  iyy="1.1192413e-05" iyz="-1.4400107e-11"

Commit message: [Fix] inertia value

File: pir2_description/urdf/body/bottom.urdf.xacro (robot description, xacro)
@@ -24,8 +24,8 @@
       <inertial>
         <origin xyz="0 0 0" rpy="0 0 0"/>
-        <mass value="1.3729096e+00"/>
-        <inertia ixx="8.7002718e-03" ixy="-4.7576583e-05" ixz="1.1160499e-04"
-                 iyy="8.6195418e-03" iyz="-3.5422299e-06"
-                 izz="1.4612727e-02" />
+        <mass value="1.3"/>
+        <inertia ixx="0.01" ixy="0" ixz="0"
+                 iyy="0.01" iyz="0"
+                 izz="0.02" />
       </inertial>
     </link>
@@ -47,13 +47,13 @@
         <origin xyz="0 0.001 -0.025" rpy="0 0 0"/>
         <geometry>
-          <sphere radius="0.05"/>
+          <sphere radius="0.0577"/>
         </geometry>
       </collision>
       <inertial>
         <origin xyz="0 0 0" />
-        <mass value="0.005" />
-        <inertia ixx="0.001" ixy="0.0" ixz="0.0"
-                 iyy="0.001" iyz="0.0"
-                 izz="0.001" />
+        <mass value="0.05" />
+        <inertia ixx="0.00005" ixy="0.0" ixz="0.0"
+                 iyy="0.00005" iyz="0.0"
+                 izz="0.00005" />
       </inertial>
     </link>
@@ -75,13 +75,13 @@
         <origin xyz="0 0.001 -0.025" rpy="0 0 0"/>
         <geometry>
-          <sphere radius="0.05"/>
+          <sphere radius="0.0585"/>
         </geometry>
       </collision>
       <inertial>
         <origin xyz="0 0 0" />
-        <mass value="0.005" />
-        <inertia ixx="0.001" ixy="0.0" ixz="0.0"
-                 iyy="0.001" iyz="0.0"
-                 izz="0.001" />
+        <mass value="0.05" />
+        <inertia ixx="0.00005" ixy="0.0" ixz="0.0"
+                 iyy="0.00005" iyz="0.0"
+                 izz="0.00005" />
       </inertial>
     </link>

File: pir2_description/urdf/body/lds_plate.urdf.xacro (robot description, xacro)
@@ -21,11 +21,11 @@
         </geometry>
       </collision>
-      <inertial>
+      <!-- <inertial>
         <origin xyz="0 0 0" rpy="0 0 0"/>
-        <mass value="0.50"/>
-        <inertia ixx="1e-3" ixy="0" ixz="0"
-                 iyy="1e-3" iyz="-0"
-                 izz="1e-3" />
-      </inertial>
+        <mass value="0.114"/>
+        <inertia ixx="0.019" ixy="0" ixz="0"
+                 iyy="0.019" iyz="-0"
+                 izz="0.004" />
+      </inertial> -->
     </link>
   </xacro:macro>

File: pir2_description/urdf/body/middle.urdf.xacro (robot description, xacro)
@@ -21,11 +21,11 @@
         </geometry>
       </collision>
-      <inertial>
+      <!-- <inertial>
         <origin xyz="0 0 0" rpy="0 0 0"/>
-        <mass value="0.50"/>
-        <inertia ixx="1e-3" ixy="0" ixz="0"
-                 iyy="1e-3" iyz="0"
-                 izz="1e-3" />
-      </inertial>
+        <mass value="0.4"/>
+        <inertia ixx="0.008" ixy="0" ixz="0"
+                 iyy="0.008" iyz="0"
+                 izz="0.016" />
+      </inertial> -->
     </link>
   </xacro:macro>

File: pir2_description/urdf/lds/lds.urdf.xacro (robot description, xacro)
@@ -22,5 +22,5 @@
         </geometry>
       </collision>
-      <inertial>
+      <!-- <inertial>
         <mass value="0.114" />
         <origin xyz="0 0 0" />
@@ -28,5 +28,5 @@
                  iyy="0.001" iyz="0.0"
                  izz="0.001" />
-      </inertial>
+      </inertial> -->
     </link>
   </xacro:macro>

File: pir2_description/urdf/wheels/wheel.urdf.xacro (robot description, xacro)
@@ -25,8 +25,8 @@
       <inertial>
         <origin xyz="0 0 0" />
-        <mass value="0.230446843750" />
-        <inertia ixx="1" ixy="0" ixz="0"
-                 iyy="1" iyz="0"
-                 izz="1" />
+        <mass value="0.22" />
+        <inertia ixx="0.0011" ixy="0" ixz="0"
+                 iyy="0.0011" iyz="0"
+                 izz="0.0017" />
         </inertial>
     </link>
@@ -53,8 +53,8 @@
       <inertial>
         <origin xyz="0 0 0" />
-        <mass value="2" />
-        <inertia ixx="1" ixy="0" ixz="0"
-                 iyy="1" iyz="0"
-                 izz="1" />
+        <mass value="0.22" />
+        <inertia ixx="0.0011" ixy="0" ixz="0"
+                 iyy="0.0011" iyz="0"
+                 izz="0.0017" />
         </inertial>
     </link>

Commit message: [Edit] inertia value

File: pir2_description/urdf/body/bottom.urdf.xacro (robot description, xacro)
@@ -23,9 +23,9 @@
       </collision>
       <inertial>
-        <origin xyz="0 0 0.275" rpy="0 0 0"/>
+        <origin xyz="0 0 0.175" rpy="0 0 0"/>
         <mass value="3.0"/>
-        <inertia ixx="0.31" ixy="0" ixz="0"
-                 iyy="0.31" iyz="0"
-                 izz="0.45" />
+        <inertia ixx="0.10" ixy="0" ixz="0"
+                 iyy="0.10" iyz="0"
+                 izz="0.20" />
       </inertial>
     </link>
@@ -47,13 +47,13 @@
         <origin xyz="0 0.001 -0.025" rpy="0 0 0"/>
         <geometry>
-          <sphere radius="0.0577"/>
+          <sphere radius="0.0588"/>
         </geometry>
       </collision>
       <inertial>
         <origin xyz="0 0 0" />
-        <mass value="0.05" />
-        <inertia ixx="0.00005" ixy="0.0" ixz="0.0"
-                 iyy="0.00005" iyz="0.0"
-                 izz="0.00005" />
+        <mass value="0.5" />
+        <inertia ixx="0.00064" ixy="0.0" ixz="0.0"
+                 iyy="0.00064" iyz="0.0"
+                 izz="0.00064" />
       </inertial>
     </link>
@@ -75,13 +75,13 @@
         <origin xyz="0 0.001 -0.025" rpy="0 0 0"/>
         <geometry>
-          <sphere radius="0.0585"/>
+          <sphere radius="0.0588"/>
         </geometry>
       </collision>
       <inertial>
         <origin xyz="0 0 0" />
-        <mass value="0.05" />
-        <inertia ixx="0.00005" ixy="0.0" ixz="0.0"
-                 iyy="0.00005" iyz="0.0"
-                 izz="0.00005" />
+        <mass value="0.5" />
+        <inertia ixx="0.00064" ixy="0.0" ixz="0.0"
+                 iyy="0.00064" iyz="0.0"
+                 izz="0.00064" />
       </inertial>
     </link>

File: pir2_description/urdf/body/middle.urdf.xacro (robot description, xacro)
@@ -21,5 +21,5 @@
         </geometry>
       </collision>
-      <!-- <inertial>
+      <inertial>
         <origin xyz="0 0 0" rpy="0 0 0"/>
         <mass value="0.8"/>
@@ -27,5 +27,5 @@
                  iyy="0.008" iyz="0"
                  izz="0.016" />
-      </inertial> -->
+      </inertial>
     </link>
   </xacro:macro>

File: pir2_description/urdf/body/top.urdf.xacro (robot description, xacro)
@@ -21,5 +21,5 @@
         </geometry>
       </collision>
-      <!-- <inertial>
+      <inertial>
         <origin xyz="0 0 0" rpy="0 0 0"/>
         <mass value="0.5"/>
@@ -27,5 +27,5 @@
                  iyy="0.0024" iyz="0"
                  izz="0.0048" />
-      </inertial> -->
+      </inertial>
     </link>
   </xacro:macro>

File: pir2_description/urdf/head/head.urdf.xacro (robot description, xacro)
@@ -41,5 +41,5 @@
      <inertial>
        <origin xyz="-0.015 0 0" rpy="0 0 0"/>
-       <mass value="0.2"/>
+       <mass value="0.02"/>
        <inertia
   	    ixx="0.0001" ixy="0.0" ixz="0.0"
@@ -73,5 +73,5 @@
       <inertial>
         <origin xyz="0 0 0.018" rpy="0 0 0"/>
-        <mass value="0.3"/>
+        <mass value="0.03"/>
         <inertia
           ixx="0.0000625" ixy="0.0" ixz="0.0"
@@ -104,5 +104,5 @@
       <inertial>
         <origin xyz="0.035 0 -0.025" rpy="0 0 0"/>
-        <mass value="0.4"/>
+        <mass value="0.04"/>
         <inertia
           ixx="0.032" ixy="0.0" ixz="0.0"
@@ -132,5 +132,5 @@
       <inertial>
         <origin xyz="-0.013 0 -0.015" rpy="0 0 0"/>
-        <mass value="0.2"/>
+        <mass value="0.02"/>
         <inertia
          ixx="0.0028" ixy="0.0" ixz="0.0"
@@ -164,5 +164,5 @@
       <inertial>
         <origin xyz="0 0 0" rpy="0 0 0"/>
-        <mass value="0.1"/>
+        <mass value="0.01"/>
         <inertia
           ixx="0.00057" ixy="0.0" ixz="0.0"

File: pir2_description/urdf/wheels/wheel.gazebo.xacro (robot description, xacro)
@@ -39,5 +39,5 @@
       <wheelDiameter>0.216</wheelDiameter>
       <wheelAcceleration>1</wheelAcceleration>
-      <wheelTorque>10</wheelTorque>
+      <wheelTorque>10000</wheelTorque>
       <rosDebugLevel>na</rosDebugLevel>
     </plugin>
