Commit message: [Edit] mass value

File: pir2_description/urdf/body/bottom.urdf.xacro (robot description, xacro)
@@ -23,9 +23,9 @@
       </collision>
       <inertial>
-        <origin xyz="0 0 0.175" rpy="0 0 0"/>
-        <mass value="3.0"/>
-        <inertia ixx="0.10" ixy="0" ixz="0"
-                 iyy="0.10" iyz="0"
-                 izz="0.20" />
+        <origin xyz="0 0 0.75" rpy="0 0 0"/>
+        <mass value="20.0"/>
+        <inertia ixx="0.24" ixy="0" ixz="0"
+                 iyy="0.24" iyz="0"
+                 izz="0.48" />
       </inertial>
     </link>
@@ -47,5 +47,5 @@
         <origin xyz="0 0.001 -0.025" rpy="0 0 0"/>
         <geometry>
-          <sphere radius="0.0588"/>
+          <sphere radius="0.056"/>
         </geometry>
       </collision>
@@ -75,5 +75,5 @@
         <origin xyz="0 0.001 -0.025" rpy="0 0 0"/>
         <geometry>
-          <sphere radius="0.0588"/>
+          <sphere radius="0.054"/>
         </geometry>
       </collision>

Commit message: [Edit] inartia point

File: pir2_description/urdf/body/bottom.urdf.xacro (robot description, xacro)
@@ -24,5 +24,5 @@
       </collision>
       <inertial>
-        <origin xyz="0 0 0.75" rpy="0 0 0"/>
+        <origin xyz="0 0 0" rpy="0 0 0"/>
         <mass value="20.0"/>
         <inertia ixx="0.24" ixy="0" ixz="0"
