Commit message: [Edit] ineratia value

File: pir2_description/robots/pir2_base_frame.urdf.xacro (robot description, xacro)
@@ -9,5 +9,4 @@
   <xacro:include filename="$(find pir2_description)/urdf/wheels/wheel.urdf.xacro"/>
   <xacro:include filename="$(find pir2_description)/urdf/lds/lds.urdf.xacro"/>
-  <xacro:include filename="$(find pir2_description)/urdf/head/head.urdf.xacro"/>
   <xacro:bottom_frame parent="base_footprint"/>
   <xacro:middle_frame parent="base_link"/>
@@ -16,7 +15,4 @@
   <xacro:lds parent="lds_plate_link" />
   <xacro:wheel parent="base_link" />
-  <xacro:head_frame parent="top_link" angle="1.0471975511965976" />
-  <xacro:head_frame_transmission />
-  <xacro:head_frame_gazebo />
   <!-- =============== Gazebo =============== -->
   <gazebo>

File: pir2_description/urdf/body/bottom.gazebo.xacro (robot description, xacro)
@@ -2,5 +2,27 @@
 <robot name="pir2_sim" xmlns:xacro="http://ros.org/wiki/xacro">
   <gazebo reference="base_link">
-    <material>Gazebo/DarkGrey</material>
+    <material>DarkGrey</material>
+  </gazebo>
+  <gazebo>
+    <plugin name="pir2_controller" filename="libgazebo_ros_diff_drive.so">
+      <commandTopic>cmd_vel</commandTopic>
+      <odometryTopic>odom</odometryTopic>
+      <odometryFrame>odom</odometryFrame>
+      <odometrySource>world</odometrySource>
+      <publishOdomTF>true</publishOdomTF>
+      <robotBaseFrame>base_footprint</robotBaseFrame>
+      <publishWheelTF>false</publishWheelTF>
+      <publishTf>true</publishTf>
+      <publishWheelJointState>true</publishWheelJointState>
+      <legacyMode>false</legacyMode>
+      <updateRate>30</updateRate>
+      <leftJoint>wheel_left_joint</leftJoint>
+      <rightJoint>wheel_right_joint</rightJoint>
+      <wheelSeparation>0.56</wheelSeparation>
+      <wheelDiameter>0.5</wheelDiameter>
+      <wheelAcceleration>1</wheelAcceleration>
+      <wheelTorque>100</wheelTorque>
+      <rosDebugLevel>na</rosDebugLevel>
+    </plugin>
   </gazebo>
 </robot>

File: pir2_description/urdf/body/bottom.urdf.xacro (robot description, xacro)
@@ -23,9 +23,9 @@
       </collision>
       <inertial>
-        <origin xyz="0 0 0" rpy="0 0 0"/>
-        <mass value="1.3"/>
-        <inertia ixx="0.01" ixy="0" ixz="0"
-                 iyy="0.01" iyz="0"
-                 izz="0.02" />
+        <origin xyz="0 0 0.275" rpy="0 0 0"/>
+        <mass value="3.0"/>
+        <inertia ixx="0.31" ixy="0" ixz="0"
+                 iyy="0.31" iyz="0"
+                 izz="0.45" />
       </inertial>
     </link>

File: pir2_description/urdf/body/top.urdf.xacro (robot description, xacro)
@@ -23,8 +23,8 @@
       <!-- <inertial>
         <origin xyz="0 0 0" rpy="0 0 0"/>
-        <mass value="0.7"/>
-        <inertia ixx="0.0034" ixy="0" ixz="0"
-                 iyy="0.0034" iyz="0"
-                 izz="0.0068" />
+        <mass value="0.5"/>
+        <inertia ixx="0.0024" ixy="0" ixz="0"
+                 iyy="0.0024" iyz="0"
+                 izz="0.0048" />
       </inertial> -->
     </link>
