Commit message: [Add] yaw joint

File: pir2_description/robots/pir2_frame.urdf.xacro (robot description, xacro)
@@ -16,4 +16,6 @@
   <xacro:wheel parent="base_link" />
   <xacro:head_frame parent="top_link" />
+  <xacro:head_frame_transmission />
+  <xacro:head_frame_gazebo />
   <!-- =============== Gazebo =============== -->
   <gazebo>

File: pir2_description/urdf/head/head.urdf.xacro (robot description, xacro)
@@ -1,7 +1,8 @@
 <?xml version="1.0"?>
 <robot name="head_base_frame" xmlns:xacro="http://www.ros.org/wiki/xacro">
-  <!--xacro:include filename="$(find pir2_description)/urdf/head/head.transmission.xacro"/-->
-  <!--xacro:include filename="$(find pir2_description)/urdf/head/head.gazebo.xacro"/-->
+  <xacro:include filename="$(find pir2_description)/urdf/head/head.transmission.xacro"/>
+  <xacro:include filename="$(find pir2_description)/urdf/head/head.gazebo.xacro"/>
   <xacro:macro name="head_frame" params="parent">
+    <xacro:property name="yaw_angle" value="0"/>
     <joint name="head_base_joint" type="fixed">
       <origin xyz="0 0 0.0316 " rpy="0 0 0" />
@@ -53,4 +54,79 @@
      </inertial>
     </link>
+    <joint name="tilt_joint" type="revolute">
+      <parent link="pan_link"/>
+      <child link="tilt_link"/>
+      <origin xyz="0 0.0245 0.0515" rpy="-1.57 -1.57 0" />
+      <axis xyz="0 0 1" />
+      <limit lower="-1.3" upper="1.3" effort="10" velocity="1"/>
+      <dynamics damping="0.7"/>
+    </joint>
+    <link name="tilt_link" >
+      <visual>
+        <origin xyz="0 0 -0.0245" rpy="0 0 0" />
+        <geometry>
+          <!--box size="0.07 0.085 0.065" /-->
+          <mesh filename="package://pir2_description/meshes/head/yaw_plate.stl" scale="0.001 0.001 0.001"/>
+        </geometry>
+        <material name="gray"/>
+      </visual>
+     <inertial>
+       <origin xyz="0 -0.0245 0" rpy="0 0 0"/>
+       <mass value="0.78"/>
+       <inertia
+      ixx="0.00190" ixy="0.0" ixz="0.0"
+      iyy="0.00202" iyz="0.0"
+      izz="0.00152"/>
+     </inertial>
+    </link>
+    <joint name="yaw_plate_to_dxl_joint" type="fixed">
+      <origin xyz="0.0233 0.1276 -0.0245" rpy="1.57 0 ${yaw_angle+1.57}" />
+      <parent link="tilt_link"/>
+      <child link="yaw_dxl_link"/>
+    </joint>
+    <link name="yaw_dxl_link" >
+      <visual>
+        <origin xyz="0 0 0" rpy="0 0 0" />
+        <geometry>
+          <!--box size="0.07 0.085 0.065" /-->
+          <mesh filename="package://pir2_description/meshes/head/yaw_frame.stl" scale="0.001 0.001 0.001"/>
+        </geometry>
+        <material name="gray"/>
+      </visual>
+     <inertial>
+       <origin xyz="0 -0.0245 0" rpy="0 0 0"/>
+       <mass value="0.78"/>
+       <inertia
+      ixx="0.00190" ixy="0.0" ixz="0.0"
+      iyy="0.00202" iyz="0.0"
+      izz="0.00152"/>
+     </inertial>
+    </link>
+    <joint name="yaw_joint" type="revolute">
+      <parent link="yaw_dxl_link"/>
+      <child link="yaw_frame"/>
+      <origin xyz="0.0245 0 0" rpy="0 -1.57 3.14" />
+      <axis xyz="0 0 1" />
+      <limit lower="-1.3" upper="1.3" effort="10" velocity="1"/>
+      <dynamics damping="0.7"/>
+    </joint>
+    <link name="yaw_frame" >
+      <visual>
+        <origin xyz="0 0 0" rpy="0 0 0" />
+        <geometry>
+          <!--box size="0.07 0.085 0.065" /-->
+          <mesh filename="package://pir2_description/meshes/head/display_frame.stl" scale="0.001 0.001 0.001"/>
+        </geometry>
+        <material name="gray"/>
+      </visual>
+     <inertial>
+       <origin xyz="0 0 0" rpy="0 0 0"/>
+       <mass value="0.78"/>
+       <inertia
+      ixx="0.00190" ixy="0.0" ixz="0.0"
+      iyy="0.00202" iyz="0.0"
+      izz="0.00152"/>
+     </inertial>
+    </link>
   </xacro:macro>
 </robot>

Commit message: [Fix] head transmission and gazebo

File: pir2_description/robots/pir2_frame.urdf.xacro (robot description, xacro)
@@ -21,5 +21,5 @@
   <gazebo>
     <plugin name="gazebo_ros_control" filename="libgazebo_ros_control.so">
-      <robotNamespace>/pri2</robotNamespace>
+      <robotNamespace>/pir2</robotNamespace>
       <robotSimType>gazebo_ros_control/DefaultRobotHWSim</robotSimType>
       <legacyModeNS>true</legacyModeNS>

File: pir2_description/urdf/head/head.gazebo.xacro (robot description, xacro)
@@ -17,5 +17,5 @@
     <material>Gazebo/LightGrey</material>
   </gazebo>
-  <gazebo reference="projector_link">
+  <gazebo reference="yaw_link">
     <mu1>0.2</mu1>
     <mu2>0.2</mu2>

File: pir2_description/urdf/head/head.urdf.xacro (robot description, xacro)
@@ -105,5 +105,5 @@
     <joint name="yaw_joint" type="revolute">
       <parent link="yaw_dxl_link"/>
-      <child link="yaw_frame"/>
+      <child link="yaw_link"/>
       <origin xyz="0.0245 0 0" rpy="0 -1.57 3.14" />
       <axis xyz="0 0 1" />
@@ -111,5 +111,5 @@
       <dynamics damping="0.7"/>
     </joint>
-    <link name="yaw_frame" >
+    <link name="yaw_link" >
       <visual>
         <origin xyz="0 0 0" rpy="0 0 0" />

Commit message: [Fix] yaw angle

File: pir2_description/robots/pir2_frame.urdf.xacro (robot description, xacro)
@@ -15,5 +15,5 @@
   <xacro:lds parent="lds_plate_link" />
   <xacro:wheel parent="base_link" />
-  <xacro:head_frame parent="top_link" />
+  <xacro:head_frame parent="top_link" angle="1.0471975511965976" />
   <xacro:head_frame_transmission />
   <xacro:head_frame_gazebo />

File: pir2_description/urdf/head/head.urdf.xacro (robot description, xacro)
@@ -3,6 +3,6 @@
   <xacro:include filename="$(find pir2_description)/urdf/head/head.transmission.xacro"/>
   <xacro:include filename="$(find pir2_description)/urdf/head/head.gazebo.xacro"/>
-  <xacro:macro name="head_frame" params="parent">
-    <xacro:property name="yaw_angle" value="0"/>
+  <xacro:macro name="head_frame" params="parent angle">
+    <xacro:property name="yaw_angle" value="${-angle}"/>
     <joint name="head_base_joint" type="fixed">
       <origin xyz="0 0 0.0316 " rpy="0 0 0" />
@@ -98,5 +98,5 @@
     </link>
     <joint name="yaw_plate_to_dxl_joint" type="fixed">
-      <origin xyz="0.0233 0.1276 -0.0245" rpy="1.57 0 ${yaw_angle+1.57}" />
+      <origin xyz="0.0233 0.1 -0.0245" rpy="1.57 0 ${yaw_angle+1.57}" />
       <parent link="tilt_link"/>
       <child link="yaw_dxl_link"/>
@@ -104,5 +104,5 @@
     <link name="yaw_dxl_link" >
       <visual>
-        <origin xyz="0 0 0" rpy="0 0 0" />
+        <origin xyz="0.027 0 0" rpy="0 0 0" />
         <geometry>
           <mesh filename="package://pir2_description/meshes/head/yaw_frame.stl" scale="0.001 0.001 0.001"/>
@@ -128,5 +128,5 @@
       <parent link="yaw_dxl_link"/>
       <child link="yaw_link"/>
-      <origin xyz="0.0245 0 0" rpy="0 -1.57 3.14" />
+      <origin xyz="0.0515 0 0" rpy="0 -1.57 3.14" />
       <axis xyz="0 0 1" />
       <limit lower="-1.3" upper="1.3" effort="10" velocity="1"/>

Commit message: [Fix] from stl to dae

File: pir2_description/robots/pir2_frame.urdf.xacro (robot description, xacro)
@@ -16,5 +16,5 @@
   <xacro:lds parent="lds_plate_link" />
   <xacro:wheel parent="base_link" />
-  <xacro:head_frame parent="top_link" angle="1.0471975511965976" />
+  <xacro:head_frame parent="top_link" angle="0.5235987755982988" />
   <xacro:head_frame_transmission />
   <xacro:head_frame_gazebo />

File: pir2_description/urdf/body/bottom.gazebo.xacro (robot description, xacro)
@@ -3,4 +3,14 @@
   <gazebo reference="base_link">
     <material>LightGrey</material>
+  </gazebo>
+  <gazebo reference="caster_front_link">
+    <mu1>0.2</mu1>
+    <mu2>0.2</mu2>
+    <material>Gazebo/DarkGrey</material>
+  </gazebo>
+  <gazebo reference="caster_rear_link">
+    <mu1>0.2</mu1>
+    <mu2>0.2</mu2>
+    <material>Gazebo/DarkGrey</material>
   </gazebo>
   <gazebo>

File: pir2_description/urdf/body/bottom.urdf.xacro (robot description, xacro)
@@ -13,5 +13,5 @@
         <origin xyz="0 0 0.0" rpy="0 0 0"/>
         <geometry>
-          <mesh filename="package://pir2_description/meshes/base/bottom_frame.stl" scale="0.001 0.001 0.001"/>
+          <mesh filename="package://pir2_description/meshes/base/bottom_frame.dae" scale="0.001 0.001 0.001"/>
         </geometry>
         <material name="light_black"/>

File: pir2_description/urdf/body/lds_plate.urdf.xacro (robot description, xacro)
@@ -13,5 +13,5 @@
           <mesh filename="package://pir2_description/meshes/base/lds_frame.stl" scale="0.001 0.001 0.001"/>
         </geometry>
-        <material name="light_black"/>
+        <material name="dark"/>
       </visual>
       <collision>
@@ -29,4 +29,9 @@
       </inertial> -->
     </link>
+    <gazebo reference="lds_plate_link">
+      <mu1>0.2</mu1>
+      <mu2>0.2</mu2>
+      <material>Gazebo/DarkGrey</material>
+    </gazebo>
   </xacro:macro>
 </robot>

File: pir2_description/urdf/body/middle.urdf.xacro (robot description, xacro)
@@ -11,5 +11,5 @@
         <origin xyz="0 0 0.0" rpy="0 0 0"/>
         <geometry>
-          <mesh filename="package://pir2_description/meshes/base/middle_frame.stl" scale="0.001 0.001 0.001"/>
+          <mesh filename="package://pir2_description/meshes/base/middle_frame.dae" scale="0.001 0.001 0.001"/>
         </geometry>
         <material name="light_black"/>

File: pir2_description/urdf/body/top.urdf.xacro (robot description, xacro)
@@ -11,5 +11,5 @@
         <origin xyz="0 0 0.0" rpy="0 0 0"/>
         <geometry>
-          <mesh filename="package://pir2_description/meshes/base/top_frame.stl" scale="0.001 0.001 0.001"/>
+          <mesh filename="package://pir2_description/meshes/base/top_frame.dae" scale="0.001 0.001 0.001"/>
         </geometry>
         <material name="light_black"/>

File: pir2_description/urdf/head/head.gazebo.xacro (robot description, xacro)
@@ -10,5 +10,5 @@
     <mu1>0.2</mu1>
     <mu2>0.2</mu2>
-    <material>Gazebo/Green</material>
+    <material>Gazebo/Grey</material>
   </gazebo>
   <gazebo reference="tilt_link">

File: pir2_description/urdf/head/head.urdf.xacro (robot description, xacro)
@@ -29,5 +29,5 @@
         <geometry>
           <!--box size="0.07 0.085 0.065" /-->
-          <mesh filename="package://pir2_description/meshes/head/pan_frame.stl" scale="0.001 0.001 0.001"/>
+          <mesh filename="package://pir2_description/meshes/head/pan_frame.dae" scale="0.001 0.001 0.001"/>
         </geometry>
         <material name="grey"/>
@@ -61,5 +61,5 @@
         <geometry>
           <!--box size="0.07 0.085 0.065" /-->
-          <mesh filename="package://pir2_description/meshes/head/tilt_frame.stl" scale="0.001 0.001 0.001"/>
+          <mesh filename="package://pir2_description/meshes/head/tilt_frame.dae" scale="0.001 0.001 0.001"/>
         </geometry>
         <material name="grey"/>
@@ -92,5 +92,5 @@
         <origin xyz="0 0 -0.0245" rpy="0 0 0" />
         <geometry>
-          <mesh filename="package://pir2_description/meshes/head/yaw_plate.stl" scale="0.001 0.001 0.001"/>
+          <mesh filename="package://pir2_description/meshes/head/yaw_plate.dae" scale="0.001 0.001 0.001"/>
         </geometry>
         <material name="grey"/>
@@ -120,5 +120,5 @@
         <origin xyz="0.027 0 0" rpy="0 0 0" />
         <geometry>
-          <mesh filename="package://pir2_description/meshes/head/yaw_frame.stl" scale="0.001 0.001 0.001"/>
+          <mesh filename="package://pir2_description/meshes/head/yaw_frame.dae" scale="0.001 0.001 0.001"/>
         </geometry>
         <material name="grey"/>
@@ -154,5 +154,5 @@
           <mesh filename="package://pir2_description/meshes/head/display_frame.stl" scale="0.001 0.001 0.001"/>
         </geometry>
-        <material name="grey"/>
+        <material name="dark"/>
       </visual>
       <collision>

File: pir2_description/urdf/wheels/wheel.gazebo.xacro (robot description, xacro)
@@ -9,5 +9,5 @@
     <maxVel>0.1</maxVel>
     <fdir1>1 0 0</fdir1>
-    <material>LightGrey</material>
+    <material>Gazebo/DarkGrey</material>
   </gazebo>
   <gazebo reference="wheel_right_link">
@@ -19,5 +19,5 @@
     <maxVel>0.1</maxVel>
     <fdir1>1 0 0</fdir1>
-    <material>LightGrey</material>
+    <material>Gazebo/DarkGrey</material>
   </gazebo>
   <gazebo>
