Commit message: [Fix] limit value of tilt joint angle

File: pir2_description/urdf/head/head.urdf.xacro (robot description, xacro)
@@ -71,5 +71,5 @@
       <origin xyz="0 0.0245 0.0515" rpy="-1.57 -1.57 0" />
       <axis xyz="0 0 1" />
-      <limit lower="-1.3" upper="1.3" effort="10" velocity="1"/>
+      <limit lower="-0.3490658503988659" upper="0.17453292519943295" effort="10" velocity="1"/>
       <dynamics damping="0.7"/>
     </joint>

Commit message: [Edit] trace server

File: pir2_description/urdf/head/head.urdf.xacro (robot description, xacro)
@@ -53,5 +53,5 @@
       <origin xyz="0 0 0.0245" rpy="0 0 0" />
       <axis xyz="0 0 1" />
-      <limit lower="-1.3" upper="1.3" effort="10" velocity="1"/>
+      <limit lower="-3.14" upper="3.14" effort="10" velocity="1"/>
       <dynamics damping="0.7"/>
     </joint>
@@ -144,5 +144,5 @@
       <origin xyz="0.0515 0 0" rpy="0 -1.57 3.14" />
       <axis xyz="0 0 1" />
-      <limit lower="-1.3" upper="1.3" effort="10" velocity="1"/>
+      <limit lower="-3.4" upper="3.4" effort="10" velocity="1"/>
       <dynamics damping="0.7"/>
     </joint>

Commit message: [Fix] teleop_key node for GAZEBO

File: pir2_description/urdf/head/head.urdf.xacro (robot description, xacro)
@@ -144,5 +144,5 @@
       <origin xyz="0.0515 0 0" rpy="0 -1.57 3.14" />
       <axis xyz="0 0 1" />
-      <limit lower="-3.4" upper="3.4" effort="10" velocity="1"/>
+      <limit lower="-3.14" upper="3.14" effort="10" velocity="1"/>
       <dynamics damping="0.7"/>
     </joint>
